File: KiRA Flight Computer.kicad_pcb (KiCad board)
At the start: 4 copper layers, 85 parts, among them IC1 SC4216HSETRT, J1 Conn_01x04_Pin, J10 Conn_01x02_Pin, J2 USB_C_Receptacle_USB2.0_14P, J3 Conn_Coaxial, J4 Conn_01x03, J5 Conn_01x02, J6 Micro_SD_Card_Det1, J7 Conn_01x02_Pin, J8 Conn_01x02_Pin, J9 Conn_01x02_Pin, SW1 SW_Push, SW2 SW_SPDT, U1 ICM-426788P, U2 STM32F407VGTx, U3 MMC5883MA, U4 DPS368, U5 NEO-M9N, U6 Wio-SX1262, U7 USBLC6-2P6, U8 TPS62933P, U9 Tudi AT24CM02-SSHD-T-TUDI, Y1 16MHz 7pF, Y2 OV_7604

Commit message: Update PCB
Parts:
- added C37: 100nF, Capacitor_SMD:C_0603_1608Metric, F.Cu at (196.8, 29.0)
- C28, C29, C30, C31, C32, D2, J6, R16, R17, R5, R6, R7, R8, R9, U8, U9: moved to B.Cu
- L2: footprint dep:Inductor 60A782C -> Inductor_SMD:L_APV_APH1050; moved to B.Cu
- SW1: footprint Button_Switch_SMD:SW_Push_1P1T_NO_CK_PTS125Sx43PSMTR -> Button_Switch_SMD:SW_Push_1P1T_NO_CK_KSC6xxJ
- moved J2 171.4 mm to (42.1, 106.8), turned to 180 degrees
- moved R6 171.1 mm to (40.5, 106.8), turned to -90 degrees
- moved R5 165.7 mm to (44.0, 106.8), turned to -90 degrees
- moved J1 164.4 mm to (37.0, 117.4)
- moved C27 157.5 mm to (49.2, 107.0)
- moved U7 156.6 mm to (49.8, 110.1)
- moved C8 128.1 mm to (46.0, 124.7), turned to 135 degrees
- moved U4 126.5 mm to (44.8, 144.4)
- moved C23 126.5 mm to (40.0, 144.4)
- moved C24 126.5 mm to (42.0, 144.4)
- moved C6 125.5 mm to (47.5, 123.2), turned to 135 degrees
- moved R14 124.0 mm to (49.5, 141.5), turned to 135 degrees
- moved R15 123.5 mm to (49.2, 143.8), turned to 135 degrees
- moved C35 110.1 mm to (43.5, 155.1), turned to 90 degrees
- moved C33 109.8 mm to (46.0, 155.6), turned to 90 degrees
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Connections:
- D2 pad 1: Net-(D2-K) -> PG
- D2 pad 2: +3.3V -> Net-(D2-A)
- J1 pad 1: GND -> +3.3V
- J1 pad 2: /SWIO -> /SWCLK
- J1 pad 3: /SWCLK -> /SWIO
- J1 pad 4: +3.3V -> GND
- R10 pad 1: PG -> Net-(D2-A)
- R10 pad 2: Net-(D2-K) -> +3.3V
Routing:
- net GND: track 20.5 -> 78.4 mm, vias 0 -> 14
- net VBUS: track 1.60 -> 49.1 mm
- net +3.3V: track 33.3 -> 61.9 mm
- net /BOOT0: track 0.00 -> 28.3 mm
- net +V_REG: track 0.00 -> 26.9 mm
- net Net-(J9-Pin_2): track 0.00 -> 16.1 mm
- net /NRST: track 17.9 -> 32.0 mm, vias 0 -> 2
- net /DP+: track 0.00 -> 14.1 mm
- net I2C1_SCL: track 2.08 -> 15.9 mm
- net /DP-: track 0.00 -> 13.7 mm
- net Net-(J9-Pin_1): track 0.00 -> 12.8 mm
- net Net-(J3-In): track 0.00 -> 11.9 mm
- net I2C1_SDA: track 3.73 -> 15.3 mm
- net VREF+: track 12.0 -> 21.1 mm
- net Net-(U8-RT): track 0.00 -> 8.70 mm
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- added copper zone on F.Cu, net +3.3V
- added copper zone on F.Cu, net +5V
- added copper zone on In1.Cu, net GND
- added copper zone on F.Cu, net VBUS
Other:
- board outline added: 50 x 60 mm

Commit message: Update PCB
Parts:
- removed J7: Conn_01x02_Pin, Connector_PinHeader_2.54mm:PinHeader_1x02_P2.54mm_Vertical
- C10, C11, C13, C17, C21, C22, FB1, R18, R19, U5: moved to B.Cu
- C19: footprint Capacitor_SMD:C_0402_1005Metric -> Capacitor_SMD:C_0603_1608Metric; moved to B.Cu
- R1, R2: footprint Resistor_SMD:R_0402_1005Metric -> Resistor_SMD:R_0603_1608Metric
- moved C22 138.0 mm to (45.5, 137.2)
- moved U3 132.8 mm to (47.2, 134.2), turned to -135 degrees
- moved C21 126.9 mm to (49.8, 133.5)
- moved J3 99.3 mm to (77.0, 80.5), turned to -90 degrees
- moved J10 63.0 mm to (80.8, 131.2)
- moved R18 58.9 mm to (45.2, 127.5)
- moved R19 58.7 mm to (47.0, 124.8)
- moved J8 58.5 mm to (42.2, 124.0)
- moved J6 52.5 mm to (63.5, 72.0), turned to 0 degrees
- moved U5 33.2 mm to (158.5, 54.2), turned to 90 degrees
- moved C17 29.8 mm to (78.5, 122.8), turned to 90 degrees
- moved Y2 29.5 mm to (81.2, 123.0)
- moved C20 29.3 mm to (81.3, 119.5)
- moved R2 29.1 mm to (81.2, 126.8)
- moved C19 27.3 mm to (78.0, 126.5)
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Connections:
- J10 pad 1: UART2_TX -> UART2_RX
- J10 pad 2: UART2_RX -> UART2_TX
- U1 pad 1: SPI1_MISO -> SPI2_MISO
- U1 pad 12: SPI1_CS -> SPI2_CS
- U1 pad 13: SPI1_SCK -> SPI2_SCK
- U1 pad 14: SPI1_MOSI -> SPI2_MOSI
- U2 pad 68: UART1_TX -> unconnected-(U2-PA9-Pad68)
- U2 pad 69: UART1_RX -> unconnected-(U2-PA10-Pad69)
- U6 pad 2: SPI2_MISO -> SPI1_MISO
- U6 pad 3: SPI2_MOSI -> SPI1_MOSI
- U6 pad 4: SPI2_SCK -> SPI1_SCK
- U6 pad 6: SPI2_CS -> SPI1_CS
Routing:
- net GND: track 78.4 -> 111.7 mm, vias 14 -> 21
- net SPI1_CS: track 0.00 -> 27.5 mm
- net SPI2_SCK: track 0.00 -> 21.4 mm, vias 0 -> 2
- net SPI2_CS: track 0.00 -> 20.8 mm, vias 0 -> 2
- net SPI1_SCK: track 0.00 -> 20.8 mm, vias 0 -> 2
- net SPI1_MOSI: track 0.00 -> 18.3 mm
- net SPI1_MISO: track 0.00 -> 17.6 mm
- net I2C2_SCK: track 2.53 -> 18.9 mm, vias 0 -> 1
- net I2C2_SDA: track 2.74 -> 17.8 mm, vias 0 -> 1
- net SPI2_MISO: track 0.00 -> 13.2 mm
- net SPI2_MOSI: track 0.00 -> 12.5 mm, vias 0 -> 2
- net I2C3_SDA: track 3.13 -> 15.5 mm, vias 0 -> 1
- net I2C3_SCL: track 3.15 -> 14.1 mm, vias 0 -> 1
- net Net-(J3-In): track 11.9 -> 21.8 mm
- net SPI3_MISO: track 0.00 -> 7.56 mm, vias 0 -> 2
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
Commit message: Update PCB
Parts:
- added C38: 10uF, Capacitor_SMD:C_1206_3216Metric, F.Cu at (80.5, 95.8)
- added C39: 100nF, Capacitor_SMD:C_0603_1608Metric, F.Cu at (80.5, 93.5)
- added J11: Conn_01x03_Pin, Connector_PinHeader_2.54mm:PinHeader_1x03_P2.54mm_Vertical, F.Cu at (94.8, 91.2)
- added J12: Conn_01x03_Pin, Connector_PinHeader_2.54mm:PinHeader_1x03_P2.54mm_Vertical, F.Cu at (99.5, 91.2)
- added J13: Screw_Terminal_01x02, TerminalBlock_Phoenix:TerminalBlock_Phoenix_MPT-0,5-2-2.54_1x02_P2.54mm_Horizontal, F.Cu at (65.5, 106.2)
- added J14: Screw_Terminal_01x02, TerminalBlock_Phoenix:TerminalBlock_Phoenix_MPT-0,5-2-2.54_1x02_P2.54mm_Horizontal, F.Cu at (65.5, 99.1)
- added J7: Conn_01x03, dep:CONSMA001SMDG, F.Cu at (87.5, 56.8)
- added R20: R, Resistor_SMD:R_0402_1005Metric, B.Cu at (78.8, 81.5)
- added R21: R, Resistor_SMD:R_0402_1005Metric, B.Cu at (77.0, 70.8)
- C2, C25, C26, C37, D1, R3: moved to B.Cu
- J3: value Conn_Coaxial -> Conn_01x03_Pin; footprint Connector_Coaxial:BNC_Amphenol_B6252HB-NPP3G-50_Horizontal -> Connector_PinHeader_2.54mm:PinHeader_1x03_P2.54mm_Vertical
- J6: footprint Connector_Card:microSD_HC_Hirose_DM3BT-DSF-PEJS -> Connector_Card:microSD_HC_Hirose_DM3AT-SF-PEJM5
- J9: value Conn_01x02_Pin -> Conn_01x03_Pin; footprint Connector_PinHeader_2.54mm:PinHeader_1x02_P2.54mm_Vertical -> Connector_PinHeader_2.54mm:PinHeader_1x03_P2.54mm_Vertical
- R4: footprint Resistor_SMD:R_0402_1005Metric -> Resistor_SMD:R_0603_1608Metric; moved to B.Cu
- moved C25 114.6 mm to (92.0, 81.2), turned to -90 degrees
- moved C37 114.6 mm to (93.8, 81.2), turned to -90 degrees
- moved R4 106.9 mm to (77.2, 64.5), turned to 90 degrees
- moved C26 105.5 mm to (77.2, 68.2), turned to -90 degrees
- moved L1 96.8 mm to (86.2, 63.2)
- moved D1 95.9 mm to (85.8, 60.8), turned to 180 degrees
- moved J9 94.8 mm to (90.0, 91.2)
- moved R3 90.0 mm to (88.7, 60.8), turned to 0 degrees
- moved U5 74.7 mm to (85.8, 71.0), turned to 0 degrees
- moved C31 69.5 mm to (77.8, 97.2), turned to 0 degrees
- moved R12 63.6 mm to (94.2, 104.5)
- moved C36 63.5 mm to (100.0, 104.2)
- moved IC1 63.5 mm to (88.2, 105.6)
- moved R13 63.5 mm to (94.2, 102.4)
- moved C34 63.2 mm to (97.4, 103.8)
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Connections:
- C26 pad 1: Net-(C26-Pad1) -> Net-(U5-VCC_RF)
- J10 pad 1: UART2_RX -> UART4_RX
- J10 pad 2: UART2_TX -> UART4_TX
- J3 pad 1: Net-(J3-In) -> PWM1
- J3 pad 2: GND -> +5V
- J9 pad 1: Net-(J9-Pin_1) -> PWM2
- J9 pad 2: Net-(J9-Pin_2) -> +5V
- L1 pad 1: Net-(C26-Pad1) -> Net-(L1-Pad1)
- L1 pad 2: Net-(J3-In) -> Net-(J7-Pin_3)
- R4 pad 2: Net-(C26-Pad1) -> Net-(L1-Pad1)
- U2 pad 4: unconnected-(U2-PE5-Pad4) -> PWM3
- U2 pad 41: unconnected-(U2-PE10-Pad41) -> RF_SW1
- U2 pad 42: unconnected-(U2-PE11-Pad42) -> DIO1
- U2 pad 43: unconnected-(U2-PE12-Pad43) -> BUSY
- U2 pad 5: unconnected-(U2-PE6-Pad5) -> PWM4
- U2 pad 53: DIO1 -> unconnected-(U2-PB14-Pad53)
- U2 pad 54: BUSY -> unconnected-(U2-PB15-Pad54)
- U2 pad 55: RF_SW1 -> unconnected-(U2-PD8-Pad55)
- U2 pad 59: unconnected-(U2-PD12-Pad59) -> PWM2
- U2 pad 60: unconnected-(U2-PD13-Pad60) -> PWM1
- U5 pad 1: Net-(J9-Pin_1) -> Net-(U5-~{SAFEBOOT})
- U5 pad 11: Net-(J3-In) -> Net-(J7-Pin_3)
- U5 pad 20: UART4_RX -> UART2_RX
- U5 pad 21: UART4_TX -> UART2_TX
- U5 pad 8: Net-(J9-Pin_2) -> Net-(U5-~{RESET})
Routing:
- net GND: track 111.7 -> 161.9 mm, vias 21 -> 31
- net +3.3V: track 65.6 -> 97.2 mm, vias 4 -> 24
- net SDIO_CMD: track 0.00 -> 28.1 mm, vias 0 -> 1
- net PWM2: track 0.00 -> 26.6 mm, vias 0 -> 2
- net SDIO_CK: track 0.00 -> 26.5 mm, vias 0 -> 1
- net PWM1: track 0.00 -> 24.6 mm, vias 0 -> 2
- net Net-(J3-In): track 21.8 -> 0.00 mm
- net SDIO_D0: track 0.00 -> 19.6 mm, vias 0 -> 1
- net RF_SW1: track 0.00 -> 19.1 mm, vias 0 -> 2
- net Net-(J9-Pin_2): track 16.1 -> 0.00 mm
- net /SWCLK: track 0.00 -> 15.3 mm
- net UART4_TX: track 0.00 -> 15.0 mm, vias 0 -> 1
- net Net-(J7-Pin_3): track 0.00 -> 14.9 mm, vias 0 -> 1
- net /SWIO: track 0.00 -> 14.6 mm
- net UART4_RX: track 0.00 -> 14.0 mm, vias 0 -> 1
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- added copper zone on In2.Cu, net +3.3V

Commit message: questionable changes
Parts:
- removed J7: Conn_01x03, dep:CONSMA001SMDG
- added BZ1: Buzzer, Buzzer_Beeper:Buzzer_CUI_CPT-9019S-SMT, B.Cu at (68.5, 85.2)
- added J15: Conn_Coaxial, Connector_Coaxial:U.FL_Hirose_U.FL-R-SMT-1_Vertical, F.Cu at (83.0, 46.0)
- added Q1: FDMA430NZ, dep:FDMA430NZ, F.Cu at (77.8, 27.9)
- added Q2: FDMA430NZ, dep:FDMA430NZ, F.Cu at (71.6, 102.4)
- added R22: 220R, Resistor_SMD:R_0402_1005Metric, F.Cu at (151.5, 54.8)
- added R23: 4.7k, Resistor_SMD:R_0603_1608Metric, F.Cu at (78.1, 23.8)
- added R24: 220R, Resistor_SMD:R_0402_1005Metric, F.Cu at (149.0, 40.5)
- added R25: 4.7k, Resistor_SMD:R_0603_1608Metric, B.Cu at (70.7, 104.3)
- added R26: 1R, Resistor_SMD:R_0603_1608Metric, F.Cu at (78.2, 31.3)
- added R27: 1R, Resistor_SMD:R_0603_1608Metric, F.Cu at (71.0, 106.5)
- C25, C26, D1, R16, R17, R20, R21, R3, R4, U5: moved to F.Cu
- C37: value 100nF -> 1uF; moved to F.Cu
- U6: moved to B.Cu
- moved J13 82.0 mm to (85.8, 26.8), turned to 180 degrees
- moved R21 52.5 mm to (122.3, 44.2), turned to 0 degrees
- moved R20 49.5 mm to (120.5, 55.0)
- moved J8 42.2 mm to (107.8, 89.5)
- moved C37 36.0 mm to (64.0, 61.0), turned to 180 degrees
- moved U6 34.2 mm to (69.0, 50.4)
- moved R19 34.0 mm to (104.8, 88.2)
- moved R3 33.5 mm to (109.5, 34.5), turned to 180 degrees
- moved R18 33.3 mm to (102.8, 90.0), turned to -90 degrees
- moved C25 31.8 mm to (67.5, 61.0), turned to 0 degrees
- moved J1 28.8 mm to (39.0, 52.9)
- moved U5 25.4 mm to (69.0, 51.9), turned to 180 degrees
- moved SW2 24.9 mm to (120.6, 69.2), turned to 180 degrees
- moved R11 22.3 mm to (63.2, 76.0), turned to 180 degrees
- moved R1 22.3 mm to (119.8, 75.5), turned to 180 degrees
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Connections:
- C26 pad 1: Net-(U5-VCC_RF) -> Net-(C26-Pad1)
- J13 pad 1: unconnected-(J13-Pin_1-Pad1) -> +BATT
- J13 pad 2: unconnected-(J13-Pin_2-Pad2) -> Net-(J13-Pin_2)
- J14 pad 1: unconnected-(J14-Pin_1-Pad1) -> +BATT
- J14 pad 2: unconnected-(J14-Pin_2-Pad2) -> Net-(J14-Pin_2)
- L1 pad 1: Net-(L1-Pad1) -> Net-(C26-Pad1)
- R4 pad 2: Net-(L1-Pad1) -> Net-(C26-Pad1)
- U2 pad 56: BUZZER -> unconnected-(U2-PD9-Pad56)
- U2 pad 88: unconnected-(U2-PD7-Pad88) -> BUZZER
Routing:
- net SPI1_CS: track 27.5 -> 0.00 mm
- net BUZZER: track 0.00 -> 22.3 mm, vias 0 -> 1
- net SPI1_SCK: track 20.8 -> 0.00 mm, vias 2 -> 0
- net I2C2_SCK: track 28.2 -> 8.94 mm, vias 2 -> 1
- net RF_SW1: track 19.1 -> 0.00 mm, vias 2 -> 0
- net I2C3_SDA: track 19.1 -> 0.00 mm, vias 2 -> 0
- net SPI1_MOSI: track 18.3 -> 0.00 mm
- net Net-(D1-A): track 17.8 -> 0.00 mm
- net I2C3_SCL: track 15.5 -> 0.00 mm, vias 2 -> 0
- net GND: track 161.9 -> 146.4 mm, vias 31 -> 34
- net /SWCLK: track 15.3 -> 0.00 mm
- net /SWIO: track 14.6 -> 0.00 mm
- net +3.3V: track 97.2 -> 85.5 mm, vias 24 -> 21
- net VBUS: track 41.7 -> 30.4 mm
- net BUSY: track 10.9 -> 0.00 mm
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- added copper zone on B.Cu, net +V_REG
- added copper zone on F.Cu, net GND
Other:
- board size 50 x 60 mm -> 50 x 70 mm

Commit message: PCB Update
Parts:
- added C40: 100nF, Capacitor_SMD:C_0603_1608Metric, F.Cu at (104.8, 57.5)
- added C41: 100nF, Capacitor_SMD:C_0603_1608Metric, F.Cu at (102.0, 53.0)
- added H1: MountingHole, MountingHole:MountingHole_2.2mm_M2_DIN965_Pad, F.Cu at (63.8, 40.8)
- added H2: MountingHole, MountingHole:MountingHole_2.2mm_M2_DIN965_Pad, F.Cu at (108.2, 40.8)
- added H3: MountingHole, MountingHole:MountingHole_2.2mm_M2_DIN965_Pad, F.Cu at (63.8, 110.0)
- added H4: MountingHole, MountingHole:MountingHole_2.2mm_M2_DIN965_Pad, F.Cu at (108.2, 110.0)
- added R28: 10k, Resistor_SMD:R_0603_1608Metric, F.Cu at (98.5, 53.0)
- added R29: 10k, Resistor_SMD:R_0603_1608Metric, F.Cu at (104.8, 53.2)
- added U10: BNO055, Package_LGA:LGA-28_5.2x3.8mm_P0.5mm, F.Cu at (100.5, 56.3)
- C21, C22, D2, R25, U9: moved to F.Cu
- R10, R21: moved to B.Cu
- moved R22 76.7 mm to (81.9, 86.9), turned to -135 degrees
- moved R24 62.1 mm to (92.4, 66.1), turned to 45 degrees
- moved R21 44.3 mm to (78.2, 49.5)
- moved R20 41.3 mm to (79.5, 60.0), turned to 0 degrees
- moved R1 39.4 mm to (88.2, 52.0), turned to -90 degrees
- moved R3 38.4 mm to (79.5, 58.5)
- moved SW2 36.7 mm to (93.2, 44.8)
- moved C22 36.0 mm to (103.8, 62.8), turned to -45 degrees
- moved J1 35.1 mm to (72.6, 63.2), turned to 90 degrees
- moved R23 32.4 mm to (96.8, 50.2), turned to 180 degrees
- moved U3 31.8 mm to (100.2, 64.0), turned to 45 degrees
- moved Q1 31.2 mm to (100.8, 48.8)
- moved J13 30.7 mm to (107.0, 49.0), turned to 90 degrees
- moved R26 26.7 mm to (101.2, 44.8)
- moved C21 26.5 mm to (98.8, 67.0), turned to -45 degrees
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Connections:
- net /MPU_CLK renamed /IMUs/MPU_CLK
- net Net-(Q1-D_1) renamed /Pinout/PYOUT1
- net Net-(Q2-D_1) renamed /Pinout/PYOUT2
- C7 pad 1: +3.3V -> unconnected-(C7-Pad1)
- D2 pad 1: PG -> Net-(D2-K)
- D2 pad 2: Net-(D2-A) -> +3.3V
- J13 pad 1: +BATT -> +BAT
- J14 pad 1: +BATT -> +BAT
- R10 pad 1: Net-(D2-A) -> Net-(U8-PG)
- R10 pad 2: +3.3V -> Net-(D2-K)
- U2 pad 41: RF_SW1 -> unconnected-(U2-PE10-Pad41)
- U2 pad 42: DIO1 -> unconnected-(U2-PE11-Pad42)
- U2 pad 43: BUSY -> PY1
- U2 pad 44: PG -> unconnected-(U2-PE13-Pad44)
- U2 pad 53: unconnected-(U2-PB14-Pad53) -> BUSY
- U2 pad 54: unconnected-(U2-PB15-Pad54) -> DIO1
- U2 pad 55: unconnected-(U2-PD8-Pad55) -> UART3_TX
- U2 pad 56: unconnected-(U2-PD9-Pad56) -> UART3_RX
- U2 pad 57: unconnected-(U2-PD10-Pad57) -> RF_SW1
- U2 pad 63: unconnected-(U2-PC6-Pad63) -> RX
- U2 pad 64: unconnected-(U2-PC7-Pad64) -> TX
- U2 pad 98: unconnected-(U2-PE1-Pad98) -> PY2
- U3 pad 1: SPI3_SCK -> SPI1_SCK
- U3 pad 16: SPI3_MOSI -> SPI1_MOSI
- U3 pad 4: SPI3_CS -> SPI1_CS
- U3 pad 5: SPI3_MISO -> SPI1_MISO
- U5 pad 20: UART2_RX -> UART3_RX
- U5 pad 21: UART2_TX -> UART3_TX
- U6 pad 2: SPI1_MISO -> SPI3_MISO
- U6 pad 3: SPI1_MOSI -> SPI3_MOSI
- U6 pad 4: SPI1_SCK -> SPI3_SCK
- U6 pad 6: SPI1_CS -> SPI3_CS
- U8 pad 7: PG -> Net-(U8-PG)
Routing:
- net +BAT: track 13.5 -> 121.5 mm
- net SPI3_MOSI: track 7.02 -> 46.1 mm, vias 0 -> 1
- net I2C3_SDA: track 0.00 -> 37.7 mm, vias 0 -> 1
- net I2C3_SCL: track 0.00 -> 36.3 mm, vias 0 -> 1
- net SPI3_SCK: track 6.13 -> 40.6 mm, vias 0 -> 2
- net SPI3_CS: track 5.59 -> 38.1 mm, vias 0 -> 2
- net UART3_RX: track 0.00 -> 28.1 mm, vias 0 -> 2
- net UART3_TX: track 0.00 -> 28.0 mm
- net TX: track 0.00 -> 27.7 mm, vias 0 -> 2
- net SPI3_MISO: track 7.56 -> 35.2 mm, vias 2 -> 1
- net RX: track 0.00 -> 26.6 mm, vias 0 -> 2
- net RF_SW1: track 0.00 -> 26.2 mm, vias 0 -> 1
- net Net-(Q2-G): track 0.00 -> 25.0 mm, vias 0 -> 2
- net GND: track 146.4 -> 170.0 mm, vias 34 -> 93
- net +3.3V: track 85.5 -> 107.2 mm, vias 21 -> 31
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- added copper zone on F.Cu, net /Pinout/PYOUT1
- added copper zone on F.Cu, net /Pinout/PYOUT2
- added copper zone on F.Cu, net Net-(J13-Pin_2)
- added copper zone on F.Cu, net Net-(J14-Pin_2)
Other:
- board size 50 x 70 mm -> 50 x 74.8 mm

Commit message: Silkscreen update
Routing:
- net GND: track 170.0 -> 189.9 mm, vias 93 -> 124
- net SDIO_CMD: track 28.1 -> 28.6 mm
- net SPI3_CS: vias 2 -> 1
- net +3.3V: vias 31 -> 32
- added copper zone on B.Cu, net GND
Other:
- board text added: "+"
- board text added: "3V REG"
- board text added: "5V"
- board text added: "5V REG"
- board text added: "BARO"
- board text added: "FLS"
- board text added: "GND"
- board text added: "IMU1"
- board text added: "IMU2"
- board text added: "LoRa"
- board text added: "MAG"
- board text added: "PRG SW"
- board text added: "PWM"
- board text added: "RST"
- board text added: "RX"
- board text added: "SCL"
- board text added: "SDA"
- board text added: "SRV1"
- board text added: "SRV2"
- board text added: "SRV3"
- board text added: "SRV4"
- board text added: "SWC"
- board text added: "SWIO"
- board text added: "TP"
- board text added: "TX"
- board text added: "USB - BAT"
- board text added: "USB PWR"
- board text added: "VDD"

Commit message: add dep
Routing:
- net +3.3V: track 107.2 -> 109.3 mm, vias 32 -> 33
Other:
- board text added: "PYRO1"
- board text added: "PYRO2"
Changed lines of the file:
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@@
 		)
 	)
+	(gr_text "PYRO1\n"
+		(at 110 59 90)
+		(layer "F.SilkS")
+		(effects
+			(font
+				(size 1.5 1.5)
+				(thickness 0.3)
+				(bold yes)
+			)
+			(justify left bottom)
+		)
+	)
 	(gr_text "PWM"
 		(at 102 92.5 45)
@@
 		)
 	)
+	(gr_text "PYRO2\n\n"
+		(at 66.2 113.4 0)
+		(layer "F.SilkS")
+		(effects
+			(font
+				(size 1.5 1.5)
+				(thickness 0.3)
+				(bold yes)
+			)
+			(justify left bottom)
+		)
+	)
 	(gr_text "USB - BAT\n"
 		(at 62.25 99.75 0)
@@
 	)
 	(via
+		(at 65.6 46.6)
+		(size 0.6)
+		(drill 0.3)
+		(layers "F.Cu" "B.Cu")
+		(net 2)
+	)
+	(via
 		(at 78.25 89.75)
 		(size 0.6)
@@
 	)
 	(segment
+		(start 65.58 46.58)
+		(end 65.6 46.6)
+		(width 0.25)
+		(layer "B.Cu")
+		(net 2)
+	)
+	(segment
 		(start 103.675 87.425)
 		(end 104.75 87.425)
 		(width 0.25)
 		(layer "B.Cu")
+		(net 2)
+	)
+	(segment
+		(start 63.5 46.58)
+		(end 65.58 46.58)
+		(width 0.25)
+		(layer "B.Cu")
