File: KiRA Flight Computer.kicad_pcb (KiCad board)
At the start: 4 copper layers, 50 x 74.8 mm, 112 parts, among them IC1 SC4216HSETRT, J1 Conn_01x04_Pin, J10 Conn_01x02_Pin, J11 Conn_01x03_Pin, J12 Conn_01x03_Pin, J13 Screw_Terminal_01x02, J14 Screw_Terminal_01x02, J15 Conn_Coaxial, J2 USB_C_Receptacle_USB2.0_14P, J3 Conn_01x03_Pin, J4 Conn_01x03, J5 Conn_01x02, J6 Micro_SD_Card_Det1, J8 Conn_01x02_Pin, J9 Conn_01x03_Pin, Q1 FDMA430NZ, Q2 FDMA430NZ, SW1 SW_Push, SW2 SW_SPDT, U1 ICM-426788P, U10 BNO055, U2 STM32F407VGTx, U3 MMC5883MA, U4 DPS368, U5 NEO-M9N, U6 Wio-SX1262, U7 USBLC6-2P6, U8 TPS62933P, U9 Tudi AT24CM02-SSHD-T-TUDI, Y1 16MHz 7pF, Y2 OV_7604

Commit message: update pcb
Parts:
- removed C16: 6pF, Capacitor_SMD:C_0603_1608Metric
- removed C35: 10uF, Capacitor_SMD:C_1206_3216Metric
- removed Y1: 16MHz 7pF, Crystal:Crystal_SMD_3225-4Pin_3.2x2.5mm
- added Y3: Resonator, Crystal:Resonator_SMD_Murata_CSTxExxV-3Pin_3.0x1.1mm, F.Cu at (97.2, 85.8)
- C15: value 6pF -> 100nF; moved to B.Cu
- C33, C34, C36, C38, C39, IC1, R12, R13: moved to B.Cu
- R10: moved to F.Cu
- moved C36 28.7 mm to (77.8, 86.0)
- moved C34 28.6 mm to (75.5, 85.5)
- moved C15 28.5 mm to (76.0, 104.2)
- moved R12 23.8 mm to (75.5, 89.8), turned to 90 degrees
- moved IC1 23.8 mm to (70.5, 89.8)
- moved C33 21.6 mm to (65.0, 90.9)
- moved R13 21.0 mm to (77.6, 89.5), turned to -90 degrees
- moved C38 16.4 mm to (64.3, 93.1)
- moved C39 16.1 mm to (65.0, 89.0)
- moved BZ1 11.4 mm to (77.2, 78.0), turned to 180 degrees
- moved L2 6.66 mm to (87.5, 106.4)
- moved C31 6.43 mm to (78.8, 103.6), turned to 90 degrees
- moved C32 6.00 mm to (95.5, 105.6)
- moved R7 4.01 mm to (96.5, 99.2)
- moved R11 3.75 mm to (67.0, 76.0), turned to 0 degrees
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Connections:
- C15 pad 1: RCC IN -> +V_REG
- C7 pad 1: unconnected-(C7-Pad1) -> +3.3V
Routing:
- net +3.3V: track 109.3 -> 134.2 mm, vias 33 -> 41
- net GND: track 189.9 -> 166.4 mm, vias 124 -> 331
- net BUZZER: track 21.8 -> 4.25 mm
- net +BAT: track 121.5 -> 105.4 mm
- net +V_REG: track 22.2 -> 13.9 mm, vias 0 -> 2
- net Net-(U8-PG): track 7.50 -> 14.0 mm, vias 0 -> 1
- net Net-(U8-RT): track 8.70 -> 2.43 mm
- net RCC OUT: track 13.3 -> 7.67 mm
- net Net-(D2-K): track 6.41 -> 1.95 mm, vias 1 -> 0
- net SPI3_MOSI: track 46.1 -> 42.7 mm
- net Net-(U8-SW): track 6.77 -> 3.41 mm
- net RCC IN: track 9.99 -> 7.46 mm
- net Net-(Y2-OE): track 0.00 -> 2.19 mm
- net UART4_RX: track 14.2 -> 16.3 mm
- net Net-(Q2-G): track 25.0 -> 26.6 mm
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- added copper zone on B.Cu, net +3.3V
- added copper zone on B.Cu, net +5V
- added copper zone on B.Cu, net +BAT
- added copper zone on In2.Cu, net +BAT
- added copper zone on B.Cu, net Net-(U8-SW)
Other:
- board text added: "3V LDO"
- board text added: "5V OUT"
- board text added: "BUZZER"
- board text added: "Computer"
- board text added: "Flight"
- board text added: "KiRA"
- board text added: "VDD IN"
- board text removed: "5V REG"

Commit message: Update Formulars
Parts:
- R8: value 52k -> 56k
- R9: value 10k -> 11k
Routing:
- net +3.3V: track 134.2 -> 131.9 mm, vias 41 -> 42
- net GND: track 166.4 -> 165.7 mm, vias 331 -> 363
- added copper zone on In2.Cu, net GND
