File: KiRA Flight Computer.kicad_sch (KiCad schematic)
At the start: 37 parts, among them J1 Conn_01x04_Pin, J2 USB_C_Receptacle_USB2.0_14P, SW1 SW_Push, SW2 SW_SPDT, U2 STM32F407VGTx, U3 MMC5883MA, U4 DPS368, U6 Wio-SX1262, U7 USBLC6-2P6, Y1 16MHz 7pF

Commit message: Fix
- Add decoupling cap
- Component layout
- Redraw zones
- New buck converter
- Layout tweaks
- Change connector
Parts:
- removed C12: 100nF, Capacitor_SMD:C_0603_1608Metric, symbol Device:C
- removed J1: Conn_01x04_Pin, Connector_PinHeader_2.54mm:PinHeader_1x04_P2.54mm_Vertical, symbol Connector:Conn_01x04_Pin
- removed SW2: SW_SPDT, Button_Switch_SMD:SW_SPDT_CK_JS102011SAQN, symbol Switch:SW_SPDT
- removed Y1: 16MHz 7pF, Crystal:Crystal_SMD_3225-4Pin_3.2x2.5mm, symbol Device:Crystal_GND24
- added Y3: Resonator, Crystal:Resonator_SMD_Murata_CSTxExxV-3Pin_3.0x1.1mm, symbol Device:Resonator
- C1, C2, C3, C4, C5, C6, C7: footprint Capacitor_SMD:C_0603_1608Metric -> Capacitor_SMD:C_0402_1005Metric
- C13: value 1uF -> 100nF
- C15, C16: value 6pF -> 2.2uF; footprint Capacitor_SMD:C_0603_1608Metric -> Capacitor_SMD:C_0402_1005Metric
- C27: footprint Capacitor_SMD:C_0402_1005Metric_Pad0.74x0.62mm_HandSolder -> Capacitor_SMD:C_0603_1608Metric
- R1: value 10k -> 4.7k
Connections:
- net +3.3V: now also C13.1, C7.1, R1.1
- net +3.3VA: no longer C13.1
- net GND: now also Y3.2
- net NRST: now also R1.2
- net RCC IN: now also Y3.1; no longer C15.1
- net RCC OUT: now also Y3.3; no longer C16.1
- net at U2.49 (VCAP_1): now also C16.1
- net at U2.73 (VCAP_2): now also C15.1
- net BOOT0 renamed BOOT
- net BOOT: no longer R1.2
- net SWIO renamed SWDIO
Other:
- moved on the sheet: C14, C21, SW1
