File: KiRA Flight Computer.kicad_sch (KiCad schematic)
At the start: 37 parts, among them J1 Conn_01x04_Pin, J2 USB_C_Receptacle_USB2.0_14P, SW1 SW_Push, SW2 SW_SPDT, U2 STM32F407VGTx, U3 MMC5883MA, U4 DPS368, U6 Wio-SX1262, U7 USBLC6-2P6, Y1 16MHz 7pF

Commit message: update pcb
Parts:
- removed C15, C16: 6pF, Capacitor_SMD:C_0603_1608Metric, symbol Device:C
- removed Y1: 16MHz 7pF, Crystal:Crystal_SMD_3225-4Pin_3.2x2.5mm, symbol Device:Crystal_GND24
- added Y3: Resonator, Crystal:Resonator_SMD_Murata_CSTxExxV-3Pin_3.0x1.1mm, symbol Device:Resonator
Connections:
- net +3.3V: now also C7.1
- net GND: now also Y3.2
- net RCC IN: now also Y3.1
- net RCC OUT: now also Y3.3
