File: Power.kicad_sch (KiCad schematic)
At the start: 25 parts, among them IC1 SC4216HSETRT, J4 Conn_01x03, J5 Conn_01x02, U8 TPS62933P

Commit message: update pcb
Parts:
- removed C35: 10uF, Capacitor_SMD:C_1206_3216Metric, symbol Device:C
- added C15: 100nF, Capacitor_SMD:C_0603_1608Metric, symbol Device:C
Connections:
- net +V_REG: now also C15.1
- net GND: now also C15.2
Other:
- moved on the sheet: C38, C39

Commit message: Update Formulars
Parts:
- R8: value 52k -> 56k
- R9: value 10k -> 11k
Other:
- note added: "RT=(Vout-0.5)/0.5*RB"
- note added: "RT=(Vout-0.8)/0.8*RB"
Changed lines of the file:
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@@
 	(generator_version "9.0")
 	(paper "A4")
+	(text "RT=(Vout-0.5)/0.5*RB"
+		(exclude_from_sim no)
+		(at 92.202 156.21 0)
+		(effects
+			(font
+				(size 1.27 1.27)
+			)
+		)
+	)
 	(text "NC - 500MHZ\nGND - 1200MHZ"
 		(exclude_from_sim no)
@@
 		)
 	)
+	(text "RT=(Vout-0.8)/0.8*RB"
+		(exclude_from_sim no)
+		(at 111.506 110.236 0)
+		(effects
+			(font
+				(size 1.27 1.27)
+			)
+		)
+	)
 	(junction
 		(at 114.3 81.28)
@@
 			)
 		)
-		(property "Value" "10k"
+		(property "Value" "11k"
 			(at 127 106.6799 0)
 			(effects
@@
 			)
 		)
-		(property "Value" "52k"
+		(property "Value" "56k"
 			(at 127 93.9799 0)
 			(effects
